File: bs170_simple/v2/rev-/bs170_simple.kicad_pcb (KiCad board)
At the start: 2 copper layers, 38.1 x 12.7 mm, 11 parts, among them J1 Conn_01x02_Male, J2 Conn_Coaxial, J3 Conn_Coaxial, Q1 BS170F, Q2 BS170F, Q3 BS170F

Commit message: fixed SMA connector footprint in v2, rev- design.
Parts:
- J2, J3: footprint digikey-footprints:RF_SMA_BoardEdge_142-0701-801 -> Connector_Coaxial:SMA_Samtec_SMA-J-P-X-ST-EM1_EdgeMount
- moved J3 2.03 mm to (144.0, 139.7), turned to 90 degrees
- moved J2 2.03 mm to (110.0, 139.7), turned to 270 degrees
Routing:
- net Net-(C1-Pad2): track 4.54 -> 5.24 mm
- net GND: vias 164 -> 186
