File: bs170_simple/v2/rev-/bs170_simple.sch (KiCad schematic (older format))
At the start: 11 parts, among them J1 Conn_01x02_Male, J2 Conn_Coaxial, J3 Conn_Coaxial, Q1 BS170F, Q2 BS170F, Q3 BS170F

Commit message: fixed SMA connector footprint in v2, rev- design.
Parts:
- J2, J3: footprint digikey-footprints:RF_SMA_BoardEdge_142-0701-801 -> Connector_Coaxial:SMA_Samtec_SMA-J-P-X-ST-EM1_EdgeMount
Changed lines of the file:
@@
 F 0 "J2" H 2428 4888 50  0000 C CNN
 F 1 "Conn_Coaxial" H 2428 4797 50  0000 C CNN
-F 2 "digikey-footprints:RF_SMA_BoardEdge_142-0701-801" H 2500 4650 50  0001 C CNN
+F 2 "Connector_Coaxial:SMA_Samtec_SMA-J-P-X-ST-EM1_EdgeMount" H 2500 4650 50  0001 C CNN
 F 3 " ~" H 2500 4650 50  0001 C CNN
 	1    2500 4650
@@
 F 0 "J3" H 6850 3975 50  0000 L CNN
 F 1 "Conn_Coaxial" H 6850 3884 50  0000 L CNN
-F 2 "digikey-footprints:RF_SMA_BoardEdge_142-0701-801" H 6750 4000 50  0001 C CNN
+F 2 "Connector_Coaxial:SMA_Samtec_SMA-J-P-X-ST-EM1_EdgeMount" H 6750 4000 50  0001 C CNN
 F 3 " ~" H 6750 4000 50  0001 C CNN
 	1    6750 4000
