File: bs170_pushpull/v1/rev-/bs170_pushpull.kicad_pcb (KiCad board)
At the start: 2 copper layers, 41.9 x 19 mm, 31 parts, among them J1 BIAS, J10 Q1_G, J11 Q1_G, J2 TR1, J3 TR2, J4 RF_IN, J5 RF_OUT, J6 Q1_G, J7 Q1_G, J8 Q1_G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

Commit message: fixed title on bottom silkscreen, added pdf of schematic.
Other:
- board text added: "BS170 Push Pull HF Amplifier"
- board text removed: "B2170 Push Pull HF Amplifier"
